File: kicad_pcb/keyboard.kicad_pcb (KiCad board)
At the start: 2 copper layers, 341.5 x 107.6 mm, 127 parts, among them SW1 SW_PUSH, U1 ATMEGA32U4, X1 XTAL_GND

Commit message: deleting components to add pro micro
Parts:
- removed C1, C2, C3, C4, C5, C6, C7: 22pF, Capacitor_SMD:C_0805_2012Metric_Pad1.15x1.40mm_HandSolder
- removed R1, R2: 10k, Resistor_SMD:R_0805_2012Metric_Pad1.15x1.40mm_HandSolder
- removed R3, R4: 22, Resistor_SMD:R_0805_2012Metric_Pad1.15x1.40mm_HandSolder
- removed SW1: SW_PUSH, Button_Switch_SMD:SW_SPST_TL3342
- removed U1: ATMEGA32U4, Package_QFP:TQFP-44_10x10mm_P0.8mm
- removed USB1: Molex-0548190589, keyboard_parts:Molex-0548190589-Assembly
- removed X1: XTAL_GND, Crystal:Crystal_SMD_5032-4Pin_5.0x3.2mm
- moved D_SPACE10 165.4 mm to (423.4, 118.6)
- moved D_SPACE21 165.4 mm to (423.4, 137.7)
- moved D_SPACE32 165.4 mm to (423.4, 156.7)
- moved K_BACKSPACE 165.4 mm to (451.5, 137.2)
- moved K_FN 165.4 mm to (451.5, 175.3)
- moved K_QUOTE 165.4 mm to (451.5, 156.2)
- moved D_MINUS 165.4 mm to (276.7, 137.7)
- moved D_PLUS 165.4 mm to (276.7, 118.6)
- moved D_SEMIC 165.4 mm to (442.5, 151.0)
- moved D_SLASH 165.4 mm to (276.7, 156.7)
- moved D_SPACE14 165.4 mm to (244.3, 141.5)
- moved D_SPACE19 165.4 mm to (385.3, 137.7)
- moved D_SPACE23 165.4 mm to (206.2, 151.0)
- moved D_SPACE25 165.4 mm to (244.3, 160.5)
- moved D_SPACE3 165.4 mm to (244.3, 122.4)
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Other:
- net class Default removed

Commit message: rotating alphas
Parts:
- moved D_FN 24.1 mm to (463.6, 151.8), turned to 105 degrees
- moved D_BACKSPACE 24.0 mm to (453.7, 115.0), turned to 105 degrees
- moved D_QUOTE 23.5 mm to (458.7, 133.4), turned to 105 degrees
- moved K_TAB 22.0 mm to (148.0, 117.1), turned to -15 degrees
- moved K_FN 21.5 mm to (453.8, 153.9), turned to 15 degrees
- moved K_BACKSPACE 21.5 mm to (443.9, 117.1), turned to 15 degrees
- moved K_CTRL 21.4 mm to (138.1, 153.9), turned to -15 degrees
- moved K_CAPS 21.1 mm to (143.1, 135.5), turned to -15 degrees
- moved K_QUOTE 20.9 mm to (448.9, 135.5), turned to 15 degrees
- moved D_P 19.6 mm to (433.9, 114.4), turned to 105 degrees
- moved D_TAB 19.4 mm to (157.5, 120.1), turned to 75 degrees
- moved D_SLASH1 18.9 mm to (443.7, 151.2), turned to 105 degrees
- moved D_CTRL 18.9 mm to (147.7, 156.9), turned to 75 degrees
- moved D_SEMIC 18.6 mm to (438.8, 132.8), turned to 105 degrees
- moved D_CAPS 18.5 mm to (152.6, 138.5), turned to 75 degrees
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